Commit message: 1

File: polaris_ranger_ev/model/car_model.urdf (robot description, URDF)
Before this commit: robot car_robot, 4 links, 3 joints
Links:
- removed link caster
- added link support_wheel, mass 0.5; collision sphere radius=0.1; visual sphere radius=0.1
- link chassis: mass None -> 1.14395; geometry collision box size=1.0 1.0 0.3; visual box size=1.0 1.0 0.3
- link left_wheel: mass None -> 0.5; geometry collision cylinder length=0.1 radius=0.15; visual cylinder length=0.1 radius=0.15
- link right_wheel: mass None -> 0.5; geometry collision cylinder length=0.1 radius=0.15; visual cylinder length=0.1 radius=0.15
Joints:
- removed joint caster_wheel
- removed joint left_wheel_joint
- removed joint right_wheel_joint
- added joint left_wheel2chassis: type continuous, parent chassis, child left_wheel, origin xyz=-0.4 -0.55 -0.05 rpy=-1.57 0 0, axis 0 0 1
- added joint right_wheel2chassis: type continuous, parent chassis, child right_wheel, origin xyz=-0.4 0.55 -0.05 rpy=-1.57 0 0, axis 0 0 1
- added joint support_wheel2chassis: type continuous, parent chassis, child support_wheel, origin xyz=0.4 0 -0.1 rpy=-0 0 0, axis 1 1 1
